File: controller-pcb-2025.kicad_pcb (KiCad board)
At the start: 2 copper layers, 160 x 119 mm, 37 parts, among them J1 Conn_01x02, J2 Conn_01x04, J3 Conn_01x02, J4 Conn_01x02, J5 Conn_01x02, J6 RJ45_LED_Shielded, K2 SANYOU_SRD_Form_C, SW1 SW_SPST, SW10 SW_SPST, SW11 SW_DPDT_x2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

Commit message: V2
Parts:
- added H7: MountingHole, MountingHole:MountingHole_2.7mm_M2.5, F.Cu at (143.5, 83.8)
- added H8: MountingHole, MountingHole:MountingHole_2.7mm_M2.5, F.Cu at (168.2, 97.8)
- moved J6 3.23 mm to (219.1, 58.2)
Connections:
- A1 pad D32: unconnected-(A1-PadD32) -> /ROT-SW
- A1 pad D33: unconnected-(A1-PadD33) -> /JL-SW
- A1 pad D34: unconnected-(A1-PadD34) -> /JR-SW
- SW13 pad S2: unconnected-(SW13-PadS2) -> /ROT-SW
- U2 pad 7: unconnected-(U2-SEL+-Pad7) -> VCC
- U2 pad 8: unconnected-(U2-SEL--Pad8) -> /JR-SW
- U3 pad 7: unconnected-(U3-SEL+-Pad7) -> VCC
- U3 pad 8: unconnected-(U3-SEL--Pad8) -> /JL-SW
Routing:
- net /JL-SW: track 0.00 -> 221.5 mm, vias 0 -> 2
- net /ROT-SW: track 0.00 -> 202.3 mm, vias 0 -> 1
- net /JR-SW: track 0.00 -> 129.5 mm, vias 0 -> 1
- net /RBT-TX: track 136.5 -> 137.6 mm
- net Net-(J1-Pin_2): track 201.0 -> 199.9 mm
Other:
- outline, holes or cut-outs redrawn
- board text added: "Controller PCB"
- board text added: "Game Team"
- board text added: "INPUT : 9V DO NOT LINK BACK AND FRONT FACES !!"
- board text added: "NOTICE"

Commit message: Fixes
Routing:
- net /3POS-DOWN: track 26.7 -> 32.8 mm
- net /BTN6: track 133.5 -> 135.3 mm
- net +3.3V: vias 1 -> 2

Commit message: run to fab
Parts:
- removed K2: SANYOU_SRD_Form_C, Relay_THT:Relay_SPDT_SANYOU_SRD_Series_Form_C
- added C2: 100nF, Capacitor_THT:CP_Radial_Tantal_D4.5mm_P2.50mm, F.Cu at (169.8, 151.0)
- added C3: 100nF, Capacitor_THT:CP_Radial_D4.0mm_P1.50mm, F.Cu at (111.8, 155.5)
- added D2: IN4007, Diode_THT:D_A-405_P7.62mm_Horizontal, B.Cu at (191.9, 130.0)
- added D3: IN4007, Diode_THT:D_DO-41_SOD81_P2.54mm_Vertical_AnodeUp, B.Cu at (82.3, 150.0)
- added D4: IN4007, Diode_THT:D_DO-41_SOD81_P2.54mm_Vertical_AnodeUp, F.Cu at (230.6, 147.8)
- added Q1: IRLZ44N, Package_TO_SOT_THT:TO-220-3_Horizontal_TabDown, B.Cu at (185.8, 125.7)
- added R4: 10k, Resistor_THT:R_Axial_DIN0207_L6.3mm_D2.5mm_P7.62mm_Horizontal, B.Cu at (173.6, 130.8)
- added R5: 220, Resistor_THT:R_Axial_DIN0207_L6.3mm_D2.5mm_P7.62mm_Horizontal, F.Cu at (166.2, 134.8)
- J1, J3: value Conn_01x02 -> B2B-PH; moved to F.Cu
- moved J1 2.00 mm to (80.0, 154.4), turned to 0 degrees
- moved J3 2.00 mm to (228.2, 155.2), turned to 0 degrees
Connections:
- J1 pad 1: GND -> Net-(D2-K)
- J1 pad 2: Net-(J1-Pin_2) -> +3V
- J3 pad 1: GND -> Net-(D2-K)
- J3 pad 2: Net-(J1-Pin_2) -> +3V
- U4 pad 4: GND_PWR -> GND
Routing:
- net Net-(D2-K): track 0.00 -> 201.6 mm
- net Net-(J1-Pin_2): track 199.9 -> 0.00 mm
- net +3V: track 10.6 -> 191.5 mm, vias 0 -> 2
- net GND: track 5.26 -> 89.9 mm
- net /VIBRATORS-RLY: track 39.0 -> 62.0 mm, vias 0 -> 1
- net GND_PWR: track 21.8 -> 0.00 mm
- net Net-(Q1-G): track 0.00 -> 15.7 mm
- net VCC: track 0.00 -> 15.1 mm
