File: controller-pcb-2025.kicad_sch (KiCad schematic)
At the start: 28 parts, among them J1 RJ45, J2 Conn_01x04, J3 Conn_01x02, J4 Conn_01x02, J5 Conn_01x02, SW1 SW_SPST, SW10 SW_SPST, SW11 SW_DPDT_x2, SW12 RotaryEncoder_Switch, SW2 SW_SPST, SW3 SW_SPST, SW4 SW_SPST, SW5 SW_SPST, SW6 SW_SPST, SW7 SW_SPST, SW8 SW_SPST, SW9 SW_SPST, U1 NRF24L01_Breakout, U2 COM-09032, U3 COM-09032

Commit message: V1
Parts:
- removed J1: RJ45, symbol Connector:RJ45
- removed SW12: RotaryEncoder_Switch, symbol Device:RotaryEncoder_Switch
- added H1, H2, H3, H4, H5: MountingHole, MountingHole:MountingHole_2.7mm_M2.5, symbol Mechanical:MountingHole
- added H6: MountingHole_Pad, Project:Pwr-button_LED, symbol Mechanical:MountingHole_Pad
- added J1: Conn_01x02, Connector_JST:JST_PH_B2B-PH-K_1x02_P2.00mm_Vertical, symbol Connector_Generic:Conn_01x02
- added J6: RJ45_LED_Shielded, Project:RJ45_Cetus_J1B1211CCD_Horizontal-3D-model, symbol Connector:RJ45_LED_Shielded
- added K2: SANYOU_SRD_Form_C, Relay_THT:Relay_SPDT_SANYOU_SRD_Series_Form_C, symbol Relay:SANYOU_SRD_Form_C
- added SW13: RotaryEncoder_Switch_MP, Project:RotaryEncoder_Alps_EC11E-Switch_Vertical_H20mm-3D-model, symbol Device:RotaryEncoder_Switch_MP
- added U5: ~, Project:DFR0555, symbol Project:DFR0555
- A1: footprint PCM_arduino-library:Arduino_Mega2560_R3_Shield -> Project:Arduino_Mega2560_R3_Shield_No-MH
- D1: footprint (none) -> LED_THT:LED_D5.0mm
- J3, J4: footprint Connector_AMASS:AMASS_XT30U-F_1x02_P5.0mm_Vertical -> Connector_JST:JST_PH_B2B-PH-K_1x02_P2.00mm_Vertical
- J5: footprint (none) -> Project:AMASS_XT30UPB-M_1x02_P5.0mm_Vertical
- R1, R2, R3: footprint (none) -> Resistor_THT:R_Axial_DIN0207_L6.3mm_D2.5mm_P7.62mm_Horizontal
- RV3: footprint (none) -> Project:F2031N
- SW1, SW2, SW3, SW4, SW5, SW6, SW7, SW8, SW9: footprint (none) -> Project:ADA1502
- SW10: footprint Button_Switch_THT:SW_PUSH_6mm -> Project:ADA1502
- SW11: footprint Button_Switch_THT:SW_XKB_DM1-16UD-1 -> Project:KCD2
- U1: footprint RF_Module:nRF24L01_Breakout -> Project:nRF24L01+_Breakout
- U2, U3: footprint COM-09032:XDCR_COM-09032 -> Project:XDCR_COM-09032; symbol COM-09032:COM-09032 -> Project:COM-09032
- U4: footprint LM2596:LM2596 -> Project:LM2596; symbol LM2596:LM2596 -> Project:LM2596
Connections:
- net +3V: now also K2.1; no longer J3.2 (Pin_2), J4.2 (Pin_2)
- net +9V: now also J4.2 (Pin_2); no longer J5.2 (Pin_2)
- net ENCODER-A: now also SW13.A
- net ENCODER-B: now also SW13.B
- net GND: now also U2.3 (V-), U2.6 (H-), U3.3 (V-), U3.6 (H-), H6.1, J1.1 (Pin_1), J6.1, J6.13, SW13.C, SW13.MP, SW13.S1, U5.1; no longer J4.1 (Pin_1), U2.B2A (SEL-), U2.H3 (H-), U2.S2 (SHIELD), U2.S3 (SHIELD), U2.S4 (SHIELD), U2.V3 (V-), U3.B2A (SEL-), U3.H3 (H-), U3.S2 (SHIELD), U3.S3 (SHIELD), U3.S4 (SHIELD), U3.V3 (V-), U4.4 (OUT-)
- net JL-H: now also A1.A0, U3.4 (H); no longer A1.A10, U3.H2 (H)
- net JL-V: now also A1.A1, U3.1 (V); no longer A1.A9, U3.V2 (V)
- net JR-H: now also U2.4 (H); no longer U2.H2 (H)
- net JR-V: now also U2.1 (V); no longer U2.V2 (V)
- net RBT-RX: now also J6.7
- net RBT-TX: now also J6.8
- net VCC: now also U2.2 (V+), U2.5 (H+), U3.2 (V+), U3.5 (H+); no longer U2.H1 (H+), U2.V1 (V+), U3.H1 (H+), U3.V1 (V+)
- net VIBRATORS-RLY: now reaches A1.A2
- net VIBRATORS-RLY: now also K2.5
- net SCL: now reaches A1.SCL
- net SCL: now also J2.4 (Pin_4)
- net SDA: now reaches A1.SDA
- net SDA: now also J2.3 (Pin_3)
- net DP-CLK: no longer names the net of A1.D10
- net DP-CLK: no longer J2.4 (Pin_4)
- net DP-DIO: no longer names the net of A1.D9
- net DP-DIO: no longer J2.3 (Pin_3)
- new net: J1.2 (Pin_2), J3.2 (Pin_2), K2.3
- new net: J4.1 (Pin_1), J5.2 (Pin_2)
- new net GND_PWR: K2.2, U4.4 (OUT-)
- no-connect marks 68 -> 74
Other:
- note added: "LCD"
- note removed: "DISPLAY"
- moved on the sheet: A1, J5, RV3

Commit message: V2
Parts:
- added H7, H8: MountingHole, MountingHole:MountingHole_2.7mm_M2.5, symbol Mechanical:MountingHole
Connections:
- net VCC: now also U2.7 (SEL+), U3.7 (SEL+)
- net JL-SW: now reaches U3.8 (SEL-)
- net JL-SW: now also A1.D33
- net ROT-SW: now reaches A1.D32
- net ROT-SW: now also SW13.S2
- net JR-SW: now reaches A1.D34
- net JR-SW: now also U2.8 (SEL-)
- no-connect marks 74 -> 66
Other:
- note added: "PCB"
- note added: "PWR-BUTTON"
- note added: "PWR-BUTTON-FASTENERS"

Commit message: run to fab
Parts:
- removed K2: SANYOU_SRD_Form_C, Relay_THT:Relay_SPDT_SANYOU_SRD_Series_Form_C, symbol Relay:SANYOU_SRD_Form_C
- added C2, C3: 100nF, symbol Device:C_Polarized_Small
- added D2: IN4007, Diode_THT:D_A-405_P7.62mm_Horizontal, symbol Device:D
- added D3, D4: IN4007, symbol Device:D_Small
- added Q1: IRLZ44N, Package_TO_SOT_THT:TO-220-3_Horizontal_TabDown, symbol Transistor_FET:IRLZ44N
- added R4: 10k, Resistor_THT:R_Axial_DIN0207_L6.3mm_D2.5mm_P7.62mm_Horizontal, symbol Device:R
- added R5: 220, Resistor_THT:R_Axial_DIN0207_L6.3mm_D2.5mm_P7.62mm_Horizontal, symbol Device:R
- J1, J3: value Conn_01x02 -> B2B-PH
Connections:
- net +3V: now also J1.2 (Pin_2), J3.2 (Pin_2), D3.1 (K), D4.1 (K)
- net GND: now also C2.2, C3.2, R4.1; no longer J1.1 (Pin_1), J3.1 (Pin_1)
- net GND_PWR: now also D2.2 (A), Q1.3 (S)
- net VCC: now also C2.1, C3.1
- net VIBRATORS-RLY: now also R4.2, R5.1
- new net: Q1.1 (G), R5.2
- new net: D2.1 (K), D3.2 (A), D4.2 (A), J1.1 (Pin_1), J3.1 (Pin_1), Q1.2 (D)
- no-connect marks 66 -> 65

Commit message: update
Parts:
- C2: footprint (none) -> Capacitor_THT:CP_Radial_Tantal_D4.5mm_P2.50mm
- C3: footprint (none) -> Capacitor_THT:CP_Radial_D4.0mm_P1.50mm
- D3, D4: footprint (none) -> Diode_THT:D_DO-41_SOD81_P2.54mm_Vertical_AnodeUp
Connections:
- net GND_PWR is gone; now on net GND: D2.2 (A), Q1.3 (S), U4.4 (OUT-)
Changed lines of the file:
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@@
 	)
 	(junction
-		(at 231.14 54.61)
-		(diameter 0)
-		(color 0 0 0 0)
-	)
-	(junction
 		(at 243.84 31.75)
 		(diameter 0)
@@
 		)
 	)
-	(wire
-		(pts
-			(xy 231.14 54.61) (xy 229.87 54.61)
-		)
-		(stroke
-			(width 0)
-			(type default)
-		)
-	)
 	(bus
 		(pts
@@
 	(wire
 		(pts
-			(xy 232.41 54.61) (xy 231.14 54.61)
-		)
-		(stroke
-			(width 0)
-			(type default)
-		)
-	)
-	(wire
-		(pts
 			(xy 228.6 26.67) (xy 234.95 26.67)
 		)
@@
 			)
 		)
-		(property "Value" "GND_PWR"
+		(property "Value" "GND"
 			(at 87.63 33.0199 90)
 			(effects
@@
 			)
 		)
-		(property "Footprint" ""
+		(property "Footprint" "Capacitor_THT:CP_Radial_D4.0mm_P1.50mm"
 			(at 232.41 151.13 0)
 			(effects
@@
 	)
 	(symbol
-		(lib_id "power:PWR_FLAG")
-		(at 231.14 54.61 180)
-		(unit 1)
-		(exclude_from_sim no)
-		(in_bom yes)
-		(on_board yes)
-		(dnp no)
-		(fields_autoplaced yes)
-		(property "Reference" "#FLG04"
-			(at 231.14 56.515 0)
-			(effects
-				(font
-					(size 1.27 1.27)
-				)
-				(hide yes)
-			)
-		)
-		(property "Value" "PWR_FLAG"
-			(at 231.14 59.69 0)
-			(effects
-				(font
-					(size 1.27 1.27)
-				)
-			)
-		)
-		(property "Footprint" ""
-			(at 231.14 54.61 0)
-			(effects
-				(font
-					(size 1.27 1.27)
-				)
-				(hide yes)
-			)
-		)
-		(property "Datasheet" "~"
-			(at 231.14 54.61 0)
-			(effects
-				(font
-					(size 1.27 1.27)
-				)
-				(hide yes)
-			)
-		)
-		(property "Description" "Special symbol for telling ERC where power comes from"
-			(at 231.14 54.61 0)
-			(effects
-				(font
-					(size 1.27 1.27)
-				)
-				(hide yes)
-			)
-		)
-		(pin "1"
-		)
-		(instances
-			(project ""
-				(path "/54f3370b-b4f0-41d0-bb98-fc88779db4d9"
-					(reference "#FLG04")
-					(unit 1)
-				)
-			)
-		)
-	)
-	(symbol
 		(lib_id "Mechanical:MountingHole")
 		(at 19.05 48.26 0)
@@
 	(symbol
 		(lib_id "power:GND")
-		(at 232.41 54.61 90)
+		(at 229.87 54.61 90)
 		(unit 1)
 		(exclude_from_sim no)
@@
 		(fields_autoplaced yes)
 		(property "Reference" "#PWR022"
-			(at 238.76 54.61 0)
+			(at 236.22 54.61 0)
 			(effects
 				(font
@@
 			)
 		)
-		(property "Value" "GND_PWR"
-			(at 236.22 54.6099 90)
+		(property "Value" "GND"
+			(at 233.68 54.6099 90)
 			(effects
 				(font
@@
 		)
 		(property "Footprint" ""
-			(at 232.41 54.61 0)
+			(at 229.87 54.61 0)
 			(effects
 				(font
@@
 		)
 		(property "Datasheet" ""
-			(at 232.41 54.61 0)
+			(at 229.87 54.61 0)
 			(effects
 				(font
@@
 		)
 		(property "Description" "Power symbol creates a global label with name \"GND\" , ground"
-			(at 232.41 54.61 0)
+			(at 229.87 54.61 0)
 			(effects
 				(font
@@
 			)
 		)
-		(property "Footprint" ""
+		(property "Footprint" "Diode_THT:D_DO-41_SOD81_P2.54mm_Vertical_AnodeUp"
 			(at 134.62 44.45 90)
 			(effects
@@
 			)
 		)
-		(property "Footprint" ""
+		(property "Footprint" "Capacitor_THT:CP_Radial_Tantal_D4.5mm_P2.50mm"
 			(at 181.61 148.59 0)
 			(effects
@@
 			)
 		)
-		(property "Footprint" ""
+		(property "Footprint" "Diode_THT:D_DO-41_SOD81_P2.54mm_Vertical_AnodeUp"
 			(at 134.62 24.13 90)
 			(effects
